Commit message: Add files via upload

File: jaime/urdf/cuello.urdf (robot description, URDF)
Before this commit: robot robot_name, 5 links, 4 joints
Links:
- added link cuello_3_link; visual mesh filename=package://jaime/meshes_jaime/top_segment.stl scale=0.001 0.001 0.001
- link base_link: geometry collision box size=0.4 0.1 0.7; visual mesh filename=package://jaime/meshes_jaime/base_segment.stl scale=0.001 0.001 0.001
- link cuello_2_link: geometry visual mesh filename=package://jaime/meshes_jaime/upper_segment.stl scale=0.001 0.001 0.001
- link cuello_link: geometry visual mesh filename=package://jaime/meshes_jaime/middle_segment.stl scale=0.001 0.001 0.001
- link entre_cuello_2_link: geometry visual mesh filename=package://jaime/meshes_jaime/upper_link.stl scale=0.001 0.001 0.001
- link entre_cuello_link: geometry visual mesh filename=package://jaime/meshes_jaime/middle_link.stl scale=0.001 0.001 0.001
Joints:
- added joint quinto: type revolute, parent cuello_2_link, child cuello_3_link, origin xyz=0.063 0.0 0.138 rpy=0.0 0 0.0, axis 0 1 0, limit lower=0 upper=0.785 effort=1 velocity=2
- joint cuarto: mimic (none) -> joint=tercero multiplier=1 offset=0; origin xyz=0 0.0 0.2 rpy=0.0 0 0.0 -> xyz=0.055 0.0 0.16 rpy=0.0 0 0.0
- joint primero: origin xyz=0.15 0.0 0.6 rpy=0.0 0 0.0 -> xyz=-0.158 0.0 0.68518 rpy=0.0 0 0.0
- joint segundo: mimic (none) -> joint=primero multiplier=1 offset=0; origin xyz=0 0.0 0.3 rpy=0.0 0 0.0 -> xyz=-0.02 0.0 0.12 rpy=0.0 0 0.0
- joint tercero: origin xyz=0 0.0 0.5 rpy=0.0 0 0.0 -> xyz=0.03 0.0 0.18 rpy=0.0 0 0.0
