Commit message: Add files via upload

File: jaime/urdf/cuello.xacro (robot description, xacro)
@@ -45,6 +45,7 @@
     </collision>
     <inertial>
+      <origin rpy="0 0 0" xyz="-0.048761000000000006 0.0 0.271195"/>
       <mass value="1.6895311238439816"/>
-      <inertia ixx="0.21223169365626263" ixy="0.0" ixz="0.04500324371243572" iyy="2.2194518064627823e-10" iyz="0" izz="1.9144792220944774e-11"/>
+      <inertia ixx="0.08719578772036611" ixy="5.4784475406747093e-17" ixz="0.022449725248199624" iyy="0.09476693416632961" iyz="-2.4061783957761517e-16" izz="0.015163560157224643"/>
     </inertial>
   </link>
@@ -65,6 +66,7 @@
     </collision>
     <inertial>
+      <origin rpy="0 0 0" xyz="-0.016311 0.0 0.099931"/>
       <mass value="0.04935881321854115"/>
-      <inertia ixx="0.000629936398116401" ixy="0" ixz="0.0" iyy="0.0006163253483259048" iyz="0.0" izz="5.729401271186983e-05"/>
+      <inertia ixx="0.00013683358492508186" ixy="1.0391185824431925e-20" ixz="1.6864941381036664e-05" iyy="0.0001101218997112331" iyz="4.551194773697158e-20" izz="4.4150842757921956e-05"/>
     </inertial>
   </link>
@@ -85,6 +87,7 @@
     </collision>
     <inertial>
+      <origin rpy="0 0 0" xyz="-0.008064 0.0 0.08278"/>
       <mass value="0.32942"/>
-      <inertia ixx="0.003933593389453394" ixy="0.0" ixz="0.00010357158199955683" iyy="0.0041198946334608105" iyz="0.0" izz=" 0.00032368777783023714"/>
+      <inertia ixx="0.0016762858507607943" ixy="-4.8489364878642617e-20" ixz="-0.00011633194117814697" iyy="0.0018413198294705605" iyz="-1.2568953790911309e-19" izz="0.00030225037441020564"/>
     </inertial>
   </link>
@@ -105,6 +108,7 @@
     </collision>
     <inertial>
+      <origin rpy="0 0 0" xyz="0.034091 0.0 0.104876"/>
       <mass value="0.019952905767724887"/>
-      <inertia ixx="0.0002934457265769784" ixy="0.0" ixz="0.0" iyy="0.00031028940069271745" iyz="0.0" izz="4.627756928768699e-05"/>
+      <inertia ixx="7.401008323582294e-05" ixy="4.2619599656491147e-20" ixz="-2.1641569166888918e-05" iyy="6.762990364652787e-05" iyz="1.346217893341262e-19" izz="2.3087743207129134e-05"/>
     </inertial>
   </link>
@@ -131,6 +135,7 @@
     </collision>
     <inertial>
+      <origin rpy="0 0 0" xyz="-0.003079 9.001e-10 0.04753"/>
       <mass value="0.07524443531369857"/>
-      <inertia ixx="0.00027319929001361535" ixy="0.0" ixz="0.0" iyy="0.00031126769489640935" iyz="0.0" izz="6.044156797592207e-05"/>
+      <inertia ixx="0.00010323130575479441" ixy="-4.678798365483059e-13" ixz="-5.295549059114918e-05" iyy="0.0001405766236174683" iyz="-2.5520718357180323e-12" izz="5.971848095580196e-05"/>
     </inertial>
   </link>
@@ -151,6 +156,7 @@
     </collision>
     <inertial>
+      <origin rpy="0 0 0" xyz="-0.003079 9.001e-10 0.04753"/>
       <mass value="0.050927614310487625"/>
-      <inertia ixx="0.00017247752156394368" ixy="0.0" ixz="0.0" iyy="0.0003254742281152397" iyz="0.0" izz="0.00016065292205845016"/>
+      <inertia ixx="5.342337042769748e-05" ixy="-1.9238368188254434e-20" ixz="-5.142424748971835e-05" iyy="0.00011356719668945245" iyz="-4.589475851232928e-21" izz="6.775750723831377e-05"/>
     </inertial>
   </link>
@@ -170,6 +176,7 @@
     </collision>
     <inertial>
-      <mass value="0.1"/>
-      <inertia ixx="0.1" ixy="0.0" ixz="0.0" iyy="0.1" iyz="0.0" izz="0.1"/>
+      <origin rpy="1.414 0.785 0" xyz="0 0.6 0"/>
+      <mass value="0"/>
+      <inertia ixx= "0.00023852500001664517" ixy="0" ixz="0" iyy="0.00043338531058851275" iyz="0" izz="0.0004993545010816019"/>
     </inertial>
   </link>
@@ -216,57 +223,57 @@
     <origin xyz="0.13 0.0 0.11" rpy="0.0 0 0.0"/>
   </joint>
-  <transmission name="primero_trans">
-  <type>transmission_interface/SimpleTransmission</type>
-  <joint name="primero">
-    <hardwareInterface>hardware_interface/PositionJointInterface</hardwareInterface>
-  </joint>
-  <actuator name="primero_motor">
-    <mechanicalReduction>1</mechanicalReduction>
-    <hardwareInterface>hardware_interface/PositionJointInterface</hardwareInterface>
-  </actuator>
-  </transmission>
-  <transmission name="segundo_trans">
-  <type>transmission_interface/SimpleTransmission</type>
-  <joint name="segundo">
-    <hardwareInterface>hardware_interface/PositionJointInterface</hardwareInterface>
-  </joint>
-  <actuator name="segundo_motor">
-    <mechanicalReduction>1</mechanicalReduction>
-    <hardwareInterface>hardware_interface/PositionJointInterface</hardwareInterface>
-  </actuator>
-  </transmission>
-  <transmission name="tercero_trans">
-  <type>transmission_interface/SimpleTransmission</type>
-  <joint name="tercero">
-    <hardwareInterface>hardware_interface/PositionJointInterface</hardwareInterface>
-  </joint>
-  <actuator name="tercero_motor">
-    <mechanicalReduction>1</mechanicalReduction>
-    <hardwareInterface>hardware_interface/PositionJointInterface</hardwareInterface>
-  </actuator>
-  </transmission>
-  <transmission name="cuarto_trans">
-  <type>transmission_interface/SimpleTransmission</type>
-  <joint name="cuarto">
-    <hardwareInterface>hardware_interface/PositionJointInterface</hardwareInterface>
-  </joint>
-  <actuator name="cuarto_motor">
-    <mechanicalReduction>1</mechanicalReduction>
-    <hardwareInterface>hardware_interface/PositionJointInterface</hardwareInterface>
-  </actuator>
-  </transmission>
-  <transmission name="quinto_trans">
-  <type>transmission_interface/SimpleTransmission</type>
-  <joint name="quinto">
-    <hardwareInterface>hardware_interface/PositionJointInterface</hardwareInterface>
-  </joint>
-  <actuator name="quinto_motor">
-    <mechanicalReduction>1</mechanicalReduction>
-    <hardwareInterface>hardware_interface/PositionJointInterface</hardwareInterface>
-  </actuator>
+  <transmission name="tran1">
+    <type>transmission_interface/SimpleTransmission</type>
+    <joint name="primero">
+      <hardwareInterface>EffortJointInterface</hardwareInterface>
+    </joint>
+    <actuator name="motor1">
+      <hardwareInterface>EffortJointInterface</hardwareInterface>
+      <mechanicalReduction>1</mechanicalReduction>
+    </actuator>
+  </transmission>
+  <transmission name="tran2">
+    <type>transmission_interface/SimpleTransmission</type>
+    <joint name="segundo">
+      <hardwareInterface>EffortJointInterface</hardwareInterface>
+    </joint>
+    <actuator name="motor2">
+      <hardwareInterface>EffortJointInterface</hardwareInterface>
+      <mechanicalReduction>1</mechanicalReduction>
+    </actuator>
+  </transmission>
+  <transmission name="tran3">
+    <type>transmission_interface/SimpleTransmission</type>
+    <joint name="tercero">
+      <hardwareInterface>EffortJointInterface</hardwareInterface>
+    </joint>
+    <actuator name="motor3">
+      <hardwareInterface>EffortJointInterface</hardwareInterface>
+      <mechanicalReduction>1</mechanicalReduction>
+    </actuator>
+  </transmission>
+  <transmission name="tran4">
+    <type>transmission_interface/SimpleTransmission</type>
+    <joint name="cuarto">
+      <hardwareInterface>EffortJointInterface</hardwareInterface>
+    </joint>
+    <actuator name="motor4">
+      <hardwareInterface>EffortJointInterface</hardwareInterface>
+      <mechanicalReduction>1</mechanicalReduction>
+    </actuator>
+  </transmission>
+  <transmission name="tran5">
+    <type>transmission_interface/SimpleTransmission</type>
+    <joint name="quinto">
+      <hardwareInterface>EffortJointInterface</hardwareInterface>
+    </joint>
+    <actuator name="motor5">
+      <hardwareInterface>EffortJointInterface</hardwareInterface>
+      <mechanicalReduction>1</mechanicalReduction>
+    </actuator>
   </transmission>
   <gazebo>
     <plugin name="gazebo_ros_control" filename="libgazebo_ros_control.so">
-      <robotNamespace>/</robotNamespace>
+      <robotNamespace>/jaime</robotNamespace>
     </plugin>
   </gazebo>
